File: hardware/DSPAmp.kicad_sch (KiCad schematic)
At the start: 142 parts, among them J1 Barrel_Jack, J10 SPK3-, J11 SPK4+, J12 SPK4-, J16 NCJ6FI-V, J17 NCJ6FI-V, J18 NCJ6FI-V, J19 NCJ6FI-V, J2 NCJ6FI-V, J20 Conn_02x10_Odd_Even, J21 Conn_02x10_Odd_Even, J3 NRJ6HM-1, J4 NCJ6FI-V, J5 SPK1+, J6 SPK1-, J7 SPK2+, J8 SPK2-, J9 SPK3+, Q1 2N7000, Q2 2N7000, SW1 SW_DPDT_x2, U1 TL072, U10 OPA2134, U11 OPA2134, U12 OPA2134, U3 OPA2134, U4 ADAU1701 DSP, U5 Class D Amp, U6 Class D Amp, U7 Class D Amp, U8 Class D Amp, U9 OPA2134

Commit message: feat(hardware): finalize component selection and BOM for Mouser order
Parts:
- U2: value ~ -> LM2596 Module
- U4: value ADAU1701 DSP -> ADAU1701 DSP Module
- U5, U6, U7, U8: value Class D Amp -> TPA3118 Module
Connections:
- net VGND: no longer C3.1
- net at C2.1, R1.1, R2.1: no longer U1.3 (+)
Other:
- note added: "12V Input & Virtual Ground"
- note added: "12V to 5V DC-DC Converter"
- moved on the sheet: C1, C2, C3, C4, J1, R1, R2, U1A, U1B, U1C, U2
